File: Gateway PCB v2.kicad_pcb (KiCad board)
At the start: 4 copper layers, 85 x 41 mm, 114 parts, among them J1 Conn_Coaxial, J2 Conn_01x04_Pin, J3 Conn_02x03_Odd_Even, J4 Conn_01x03_Pin, U6 TPS7A91, U7 TLV62568ADRL, X1 TG2016SMN 32.0000M-TCGNNMB

Commit message: Fix Repo
Parts:
- removed the C28 at (79.5, 71.0)
Connections:
- R12 pad 1: GND -> FB
- R13 pad 2: GND -> FB
- U7 pad 1: GND -> FB
Routing:
- net GND: track 52.8 -> 46.2 mm
- net FB: track 0.00 -> 4.00 mm
